Commit message: 1.Uncommented the front parallel link and its mimicing joint; 2.Add front parallel link and controllers.

File: dvrk_model/MTM/mtm.urdf.xacro (robot description, xacro)
@@ -112,5 +112,5 @@
       </inertial>
     </link>
-     <!--link name="${prefix}front_parallel_link">
+     <link name="${prefix}front_parallel_link">
        <visual>
          <geometry>
@@ -127,5 +127,5 @@
          <inertia ixx="8.0" ixy="0.0" ixz="0.0" iyy="8.0" iyz="0.0" izz="8.0"/>
        </inertial>
-     </link-->
+     </link>
     <joint name="${prefix}shoulder_pitch_joint" type="revolute">
       <parent link="${prefix}outer_yaw_link"/>
@@ -149,5 +149,5 @@
       <mimic joint="${prefix}elbow_pitch_joint" multiplier="1"/>
     </joint>
-    <!--joint name="${prefix}elbow_pitch_parallel_joint" type="revolute">
+    <joint name="${prefix}elbow_pitch_parallel_joint" type="revolute">
        <parent link="${prefix}top_parallel_link"/>
        <child link="${prefix}front_parallel_link"/>
@@ -157,5 +157,5 @@
        <joint_properties damping="1.0" friction="0.0"/>
        <mimic joint="${prefix}elbow_pitch_joint" multiplier="-1"/>
-     </joint-->
+     </joint>
     <joint name="${prefix}elbow_pitch_joint" type="revolute">
       <parent link="${prefix}back_parallel_link"/>

Commit message: finish rviz setting using modified DH convension

File: dvrk_model/MTM/mtm.urdf.xacro (robot description, xacro)
@@ -38,10 +38,10 @@
       <visual>
         <geometry>
-          <mesh filename="package://dvrk_model/MTM/meshes/Top Panel.dae"/>
-        </geometry>
-      </visual>
-      <collision>
-        <geometry>
-          <mesh filename="package://dvrk_model/MTM/meshes/Top Panel.STL"/>
+          <mesh filename="package://dvrk_model/MTM/meshes/right_top_panel.STL"/>
+        </geometry>
+      </visual>
+      <collision>
+        <geometry>
+          <mesh filename="package://dvrk_model/MTM/meshes/right_top_panel.STL"/>
         </geometry>
       </collision>
@@ -57,5 +57,5 @@
       <parent link="${prefix}top_panel"/>
       <child link="${prefix}outer_yaw_link"/>
-      <origin rpy="0 0 ${PI/2}" xyz="0 0 0"/>
+      <origin rpy="0 0 0" xyz="0 0 -0.21537"/>
       <axis xyz="0 0 1"/>
       <!--rotates about z axis-->
@@ -67,10 +67,10 @@
       <visual>
         <geometry>
-          <mesh filename="package://dvrk_model/MTM/meshes/OutPitch_Shoulder.dae"/>
-        </geometry>
-      </visual>
-      <collision>
-        <geometry>
-          <mesh filename="package://dvrk_model/MTM/meshes/OutPitch_Shoulder.STL"/>
+          <mesh filename="package://dvrk_model/MTM/meshes/right_outer_yaw_link.STL"/>
+        </geometry>
+      </visual>
+      <collision>
+        <geometry>
+          <mesh filename="package://dvrk_model/MTM/meshes/right_outer_yaw_link.STL"/>
         </geometry>
       </collision>
@@ -83,10 +83,10 @@
       <visual>
         <geometry>
-          <mesh filename="package://dvrk_model/MTM/meshes/ArmParallel.dae"/>
-        </geometry>
-      </visual>
-      <collision>
-        <geometry>
-          <mesh filename="package://dvrk_model/MTM/meshes/ArmParallel.STL"/>
+          <mesh filename="package://dvrk_model/MTM/meshes/right_back_parallel_link.STL"/>
+        </geometry>
+      </visual>
+      <collision>
+        <geometry>
+          <mesh filename="package://dvrk_model/MTM/meshes/right_back_parallel_link.STL"/>
         </geometry>
       </collision>
@@ -99,10 +99,10 @@
       <visual>
         <geometry>
-          <mesh filename="package://dvrk_model/MTM/meshes/ArmParallel1.dae"/>
-        </geometry>
-      </visual>
-      <collision>
-        <geometry>
-          <mesh filename="package://dvrk_model/MTM/meshes/ArmParallel1.STL"/>
+          <mesh filename="package://dvrk_model/MTM/meshes/right_top_parallel_link.STL"/>
+        </geometry>
+      </visual>
+      <collision>
+        <geometry>
+          <mesh filename="package://dvrk_model/MTM/meshes/right_top_parallel_link.STL"/>
         </geometry>
       </collision>
@@ -115,10 +115,10 @@
        <visual>
          <geometry>
-           <mesh filename="package://dvrk_model/MTM/meshes/Link.dae"/>
+           <mesh filename="package://dvrk_model/MTM/meshes/right_front_parallel_link.STL"/>
          </geometry>
        </visual>
        <collision>
          <geometry>
-           <mesh filename="package://dvrk_model/MTM/meshes/Link.STL"/>
+           <mesh filename="package://dvrk_model/MTM/meshes/right_front_parallel_link.STL"/>
          </geometry>
        </collision>
@@ -131,5 +131,5 @@
       <parent link="${prefix}outer_yaw_link"/>
       <child link="${prefix}back_parallel_link"/>  <!-- xyz= 0 0 -.19037-->
-      <origin rpy="${-PI/2} ${-PI/2} 0" xyz="0 0 -0.19037"/>
+      <origin rpy="${-PI/2} ${PI/2} 0" xyz="0 0 0"/>
       <axis xyz="0 0 1"/>
       <!--rotates about  x axis-->
@@ -141,5 +141,5 @@
       <parent link="${prefix}back_parallel_link"/>
       <child link="${prefix}top_parallel_link"/>
-      <origin rpy="0 0 ${-PI/2}" xyz="0 0 0.065"/>
+      <origin rpy="0 0 ${PI/2}" xyz="0 0 0"/>
       <axis xyz="0 0 1"/>
       <!--rotates about  x axis-->
@@ -152,5 +152,5 @@
        <parent link="${prefix}top_parallel_link"/>
        <child link="${prefix}front_parallel_link"/>
-       <origin rpy="0 0 0" xyz=".1011 0 -0.03"/>
+       <origin rpy="0 0 ${-PI/2}" xyz="0.1011 0 0"/>
        <axis xyz="0 0 1"/>
        <limit effort="100.0" lower="${-PI/4}" upper="${PI/4}" velocity="10"/>
@@ -161,5 +161,5 @@
       <parent link="${prefix}back_parallel_link"/>
       <child link="${prefix}bottom_parallel_link"/>  <!-- xyz= -->
-      <origin rpy="0 0 ${PI/2}" xyz="-.2794 0 0"/>
+      <origin rpy="0 0 ${PI/2}" xyz="0.27967 0 0"/>
       <axis xyz="0 0 1"/>
       <!--rotates about x axis-->
@@ -171,5 +171,5 @@
       <parent link="${prefix}bottom_parallel_link"/>
       <child link="${prefix}wrist_platform_link"/>  <!-- -.348 & -.02746 defined from MTMDaVinci paper and  added -.01 from original to align, -0.02746 defined from CAD file-->
-      <origin rpy="${PI/2} 0 0" xyz="-0.3645 -0.156 0.0"/>
+      <origin rpy="${-PI/2} 0 0" xyz="0.3645 0.1506 0"/>
       <axis xyz="0 0 1"/>
       <!--rotates about z axis-->
@@ -181,10 +181,10 @@
       <visual>
         <geometry>
-          <mesh filename="package://dvrk_model/MTM/meshes/WristPlatform.dae"/>
-        </geometry>
-      </visual>
-      <collision>
-        <geometry>
-          <mesh filename="package://dvrk_model/MTM/meshes/WristPlatform.STL"/>
+          <mesh filename="package://dvrk_model/MTM/meshes/right_wrist_platform_link.STL"/>
+        </geometry>
+      </visual>
+      <collision>
+        <geometry>
+          <mesh filename="package://dvrk_model/MTM/meshes/right_wrist_platform_link.STL"/>
         </geometry>
       </collision>
@@ -199,10 +199,10 @@
       <visual>
         <geometry>
-          <mesh filename="package://dvrk_model/MTM/meshes/BottomArm.dae"/>
-        </geometry>
-      </visual>
-      <collision>
-        <geometry>
-          <mesh filename="package://dvrk_model/MTM/meshes/BottomArm.STL"/>
+          <mesh filename="package://dvrk_model/MTM/meshes/right_bottom_parallel_link.STL"/>
+        </geometry>
+      </visual>
+      <collision>
+        <geometry>
+          <mesh filename="package://dvrk_model/MTM/meshes/right_bottom_parallel_link.STL"/>
         </geometry>
       </collision>
@@ -217,5 +217,5 @@
       <parent link="${prefix}wrist_platform_link"/>
       <child link="${prefix}wrist_pitch_link"/>   <!--rpy="1.57 0 3.14159 " the num .072 & .123 are defined from CAD file -->
-      <origin rpy="${-PI/2} 0 0" xyz="0 0 0"/>
+      <origin rpy="${PI/2} 0 0" xyz="0 0 0"/>
       <axis xyz="0 0 1"/>
       <!--rotates about x axis-->
@@ -227,10 +227,10 @@
       <visual>        <!-- defined from CAD file (increased in the y dir by .005-->
         <geometry>
-          <mesh filename="package://dvrk_model/MTM/meshes/WristPitch.dae"/>
+          <mesh filename="package://dvrk_model/MTM/meshes/right_wrist_pitch_link.STL"/>
         </geometry>
       </visual>
       <collision>        <!-- defined from CAD file (increased in the y dir by .005-->
         <geometry>
-          <mesh filename="package://dvrk_model/MTM/meshes/WristPitch.STL"/>
+          <mesh filename="package://dvrk_model/MTM/meshes/right_wrist_pitch_link.STL"/>
         </geometry>
       </collision>
@@ -245,5 +245,5 @@
       <parent link="${prefix}wrist_pitch_link"/>
       <child link="${prefix}wrist_yaw_link"/>    <!--  defined from CAD file-->
-      <origin rpy="${PI/2} ${-PI/2} 0" xyz="0 0 0"/>
+      <origin rpy="${-PI/2} ${PI/2} 0" xyz="0 0 0"/>
       <axis xyz="0 0 1"/>
       <!--rotates about z axis-->
@@ -255,10 +255,10 @@
       <visual>
         <geometry>
-          <mesh filename="package://dvrk_model/MTM/meshes/WristYaw.dae"/>
-        </geometry>
-      </visual>
-      <collision>
-        <geometry>
-          <mesh filename="package://dvrk_model/MTM/meshes/WristYaw.STL"/>
+          <mesh filename="package://dvrk_model/MTM/meshes/right_wrist_yaw_link.STL"/>
+        </geometry>
+      </visual>
+      <collision>
+        <geometry>
+          <mesh filename="package://dvrk_model/MTM/meshes/right_wrist_yaw_link.STL"/>
         </geometry>
       </collision>
@@ -273,5 +273,5 @@
       <parent link="${prefix}wrist_yaw_link"/>
       <child link="${prefix}wrist_roll_link"/>  <!-- -.039 & .055 defined from CAD file-->
-      <origin rpy="${-PI/2} ${PI/2} 0" xyz="0 -.039 0"/>
+      <origin rpy="${PI/2} 0 0" xyz="0 0 0"/>
       <axis xyz="0 0 -1"/>
       <!--rotates about y axis-->
@@ -283,10 +283,10 @@
       <visual>
         <geometry>
-          <mesh filename="package://dvrk_model/MTM/meshes/WristRoll.dae"/>
-        </geometry>
-      </visual>
-      <collision>
-        <geometry>
-          <mesh filename="package://dvrk_model/MTM/meshes/WristRoll.STL"/>
+          <mesh filename="package://dvrk_model/MTM/meshes/right_wrist_roll_link.STL"/>
+        </geometry>
+      </visual>
+      <collision>
+        <geometry>
+          <mesh filename="package://dvrk_model/MTM/meshes/right_wrist_roll_link.STL"/>
         </geometry>
       </collision>
