Commit message: Wake specific adjustments

File: dvrk_description/dvrk/dvrk_launch.urdf.xacro (robot description, xacro)
@@ -7,8 +7,8 @@
 <!--xacro:include filename="$(find dvrk_description)/tool_lnd/tool_lnd.urdf.xacro"/-->
 <!--change true to specify which psm or ecm you want -->
-<property name= "ecm_num_1" value = "true" />
-<property name= "psm_num_1" value = "true" />
-<property name= "psm_num_2" value = "true" />
-<property name= "psm_num_3" value = "true"  />
+<xacro:property name= "ecm_num_1" value = "true" />
+<xacro:property name= "psm_num_1" value = "true" />
+<xacro:property name= "psm_num_2" value = "true" />
+<xacro:property name= "psm_num_3" value = "false"  />
 <xacro:suj prefix=""/>
  <xacro:if value="${ecm_num_1}">

File: dvrk_description/suj/suj.urdf.xacro (robot description, xacro)
@@ -2,6 +2,6 @@
 <robot name="suj" xmlns:xacro="http://www.ros.org/wiki/xacro">
 <xacro:macro name="suj" params="prefix">
-<property name="damping" value="0.2"/>
-<property name="friction" value="1"/>
+<xacro:property name="damping" value="0.2"/>
+<xacro:property name="friction" value="1"/>
 <link name="world"/>
 <joint name="${prefix}fixed" type="fixed">
